File: Transistor Trigger for Camera/Transistor Trigger for Camera.kicad_pcb (KiCad board)
At the start: 2 copper layers, 60 x 62.7 mm, 10 parts, among them J1 Conn_01x01_Pin, J2 Conn_01x01_Pin, J3 Conn_01x01_Pin, J4 Conn_01x01_Pin, J5 Conn_01x01_Pin, J6 Conn_01x01_Pin, Q1 2N4401, U1 74HC14N_652

Commit message: second update with new 100k resistor
Parts:
- added R2: 100k, Resistor_THT:R_Axial_DIN0207_L6.3mm_D2.5mm_P15.24mm_Horizontal, F.Cu at (107.2, 97.3)
Routing:
- net Net-(J5-Pin_1): track 14.2 -> 39.8 mm, vias 0 -> 1
- net GND: track 68.7 -> 77.6 mm

Commit message: third update with Mark and parts
Parts:
- R1: value R -> 10
- R2: value 100k -> 22k

Commit message: Final revistion changes for layout
Parts:
- added D1: D, Diode_THT:D_T-1_P10.16mm_Horizontal, F.Cu at (141.6, 107.5)
- added D2: D_Zener, Diode_THT:D_T-1_P10.16mm_Horizontal, F.Cu at (148.1, 117.6)
- moved R1 28.8 mm to (159.0, 88.1), turned to -90 degrees
- moved J2 9.18 mm to (148.4, 79.0)
- moved J6 5.43 mm to (148.4, 72.1)
- moved C1 0.20 mm to (136.5, 67.1)
Routing:
- net GND: track 77.6 -> 0.00 mm
- net Net-(D1-A): track 9.64 -> 39.7 mm
- net Net-(Q1-Pad3): track 9.33 -> 28.3 mm
- net Net-(D1-K): track 16.3 -> 32.9 mm
- net /Link_2_and_3: track 2.54 -> 14.3 mm
- net +5V: track 72.6 -> 66.3 mm
- net Net-(J5-Pin_1): track 39.8 -> 38.2 mm, vias 1 -> 0
- added copper zone on B.Cu, net GND
Other:
- board text added: "K"
- board text added: "Output"
- board text added: "Pin 1 Input"
- board text removed: "-"
- board text removed: "Pin 1 Input Tr Signal"

Commit message: further changes to layout
Routing:
- net Net-(D1-A): track 39.7 -> 46.2 mm
